Commit message: MVP

File: data/gemini.urdf (robot description, URDF)
Before this commit: robot simple_5dof_robot, 6 links, 5 joints
Links:
- link end_effector_link: geometry collision box size=0.05 0.05 0.05; visual box size=0.05 0.05 0.05
- link link_2: geometry collision box size=0.05 0.05 0.3; visual box size=0.05 0.05 0.3
- link link_3: geometry collision cylinder length=0.2 radius=0.04; visual box size=0.05 0.05 0.3
- link link_4: geometry collision cylinder length=0.15 radius=0.04; visual box size=0.05 0.05 0.3
Joints:
- joint joint_1: limit lower=-3.14 upper=3.14 effort=10 velocity=1 -> lower=-1 upper=1 effort=10 velocity=1
- joint joint_2: limit lower=-1.57 upper=1.57 effort=10 velocity=1 -> lower=-1.57 upper=.65 effort=10 velocity=1
- joint joint_3: axis 1 0 0 -> 0 0 1; limit lower=-1.57 upper=1.57 effort=10 velocity=1 -> lower=-0.57 upper=1 effort=10 velocity=1
- joint joint_4: axis 0 0 1 -> 1 0 0; limit lower=-1.57 upper=1.57 effort=10 velocity=1 -> lower=-1 upper=1 effort=10 velocity=1

Commit message: Opacity controls

File: data/gemini.urdf (robot description, URDF)
Before this commit: robot simple_5dof_robot, 6 links, 5 joints
Joints:
- joint joint_1: limit lower=-1 upper=1 effort=10 velocity=1 -> lower=0 upper=1 effort=10 velocity=1
- joint joint_2: limit lower=-1.57 upper=.65 effort=10 velocity=1 -> lower=-2.57 upper=.65 effort=10 velocity=1
